Commit message: kp160带切换

File: source/instinctlab/instinctlab/assets/resources/unitree_b2/urdf/b2rm.urdf (robot description, URDF)
Before this commit: robot b2rm, 54 links, 53 joints
Links:
- removed link si63_back_payload_link
Joints:
- removed joint si63_back_payload_joint

File: source/instinctlab/instinctlab/assets/resources/unitree_b2rm/urdf/b2rm.urdf (robot description, URDF)
Before this commit: robot b2rm, 54 links, 53 joints
Links:
- removed link si63_back_payload_link
Joints:
- removed joint si63_back_payload_joint

File: source/instinctlab/instinctlab/assets/resources/unitree_b2rm/urdf/b2rm_fast.urdf (robot description, URDF)
Before this commit: robot b2rm, 54 links, 53 joints
Links:
- removed link si63_back_payload_link
Joints:
- removed joint si63_back_payload_joint
